File: OLEDU_KiCad/OLEDUKEY/_autosave-RGB_Keys.sch (KiCad schematic (older format))
At the start: 212 parts, among them J301 Conn_01x03, J701 Conn_01x03, U301 74LVC1G125, U701 74LVC1G125

Commit message: pcb no copper
Parts:
- D301, D302, D303, D304, D305, D306, D307, D308, D309, D310, D311, D312, D313, D314, D315, D316, D317, D318, D319, D320, D321, D322, D323, D324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: footprint Keebio-Parts:SK6812-MINI-E -> LED_SDM_MOD:SK6812-MINI-E
Connections:
- wire segments 1384 -> 1395
