File: OLEDU_KiCad/OLEDUKEY/_autosave-OLEDUKEY.kicad_pcb (KiCad board)
At the start: 2 copper layers, 403.9 x 129.5 mm, 399 parts, among them J1 USB_C_TYPE-C-31-M-12, J301 Conn_01x03, J701 Conn_01x03, SW1 SW_Push, SW10 SW_Push, SW11 SW_Push, SW12 SW_Push, SW13 SW_Push, SW14 SW_Push, SW15 SW_Push, SW16 SW_Push, SW17 SW_Push, SW18 SW_Push, SW19 SW_Push, SW2 SW_Push, SW20 SW_Push, SW21 SW_Push, SW22 SW_Push, SW23 SW_Push, SW25 SW_Push, SW26 SW_Push, SW27 SW_Push, SW28 SW_Push, SW29 SW_Push, SW3 SW_Push, SW31 SW_Push, SW32 SW_Push, SW33 SW_Push, SW34 SW_Push, SW35 SW_Push, SW36 SW_Push, SW37 SW_Push, SW38 SW_Push, SW39 SW_Push, SW4 SW_Push, SW40 SW_Push, SW41 SW_Push, SW43 SW_Push, SW44 SW_Push, SW45 SW_Push, SW46 SW_Push, SW47 SW_Push, SW49 SW_Push, SW5 SW_Push, SW50 SW_Push, SW51 SW_Push, SW52 SW_Push, SW53 SW_Push, SW54 SW_Push, SW55 SW_Push, SW56 SW_Push, SW57 SW_Push, SW58 SW_Push, SW59 SW_Push, SW6 SW_Push, SW60 SW_Push, SW61 SW_Push, SW62 SW_Push, SW63 SW_Push, SW64 SW_Push, SW65 SW_Push, SW66 SW_Push, SW67 SW_Push, SW68 SW_Push, SW69 SW_Push, SW7 SW_Push, SW70 SW_Push, SW71 SW_Push, SW72 SW_Push, SW73 SW_Push, SW74 SW_Push, SW75 SW_Push, SW76 SW_Push, SW79 SW_Push, SW8 SW_Push, SW80 SW_Push, SW81 SW_Push, SW82 SW_Push, SW83 SW_Push, SW84 SW_Push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

Commit message: pcb no copper
Parts:
- D301, D302, D303, D304, D305, D306, D307, D308, D309, D310, D311, D312, D313, D314, D315, D316, D317, D318, D319, D320, D321, D322, D323, D324, D325, D326, D327, D328, D329, D330, D331, D332, D333, D334, D335, D336, D337, D338, D339, D340, D341, D342, D343, D344, D345, D346, D347, D348, D349, D350, D351, D352, D353, D354, D355, D356, D357, D358, D359, D360, D361, D362, D363, D364, D365, D366, D367, D368, D369, D370, D371, D372, D373, D374, D375, D376, D377, D378, D379, D380, D381, D382, D383, D384, D385, D386: footprint Keebio-Parts:SK6812-MINI-E -> LED_SDM_MOD:SK6812-MINI-E
- D701, D702, D703, D704, D705, D706, D707, D708, D709, D710, D711, D712, D713, D714, D715, D716, D717, D718: footprint LED_SMD:LED_SK6812MINI_PLCC4_3.5x3.5mm_P1.75mm -> LED_SDM_MOD:LED_SK6812MINI_PLCC4_3.5x3.5mm_P1.75mm
- U1: moved to F.Cu
- moved C3 83.0 mm to (344.4, 64.5)
- moved C2 72.5 mm to (297.3, 64.9)
- moved J1 43.2 mm to (320.0, -30.5)
- moved C1 40.1 mm to (329.8, 24.3)
- moved C7 38.0 mm to (304.8, -7.21), turned to 270 degrees
- moved C6 37.7 mm to (309.6, -7.21), turned to 270 degrees
- moved C5 37.6 mm to (334.0, -7.21), turned to 270 degrees
- moved C4 37.5 mm to (329.4, -7.34), turned to 270 degrees
- moved U701 17.3 mm to (328.5, 5.04), turned to 90 degrees
- moved C712 17.1 mm to (69.3, 91.6), turned to 180 degrees
- moved U301 15.7 mm to (315.1, 5.08), turned to 90 degrees
- moved R1 15.4 mm to (280.8, 38.2)
- moved C711 15.0 mm to (13.6, 91.8), turned to 180 degrees
- moved U3 14.9 mm to (320.0, -9.14)
- moved C713 14.3 mm to (131.9, 90.7), turned to 180 degrees
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Connections:
- C331 pad 1: Net-(C331-Pad1) -> USB_5v
- C332 pad 1: Net-(C331-Pad1) -> USB_5v
- C704 pad 1: Net-(C704-Pad1) -> USB_5v
- C708 pad 1: Net-(C708-Pad1) -> USB_5v
- C709 pad 1: Net-(C709-Pad1) -> USB_5v
- C710 pad 1: Net-(C710-Pad1) -> USB_5v
- C711 pad 1: Net-(C711-Pad1) -> USB_5v
- C712 pad 1: Net-(C712-Pad1) -> USB_5v
- C716 pad 1: Net-(C716-Pad1) -> USB_5v
- D1 pad 1: Net-(D1-Pad1) -> ROW0
- D10 pad 1: Net-(D10-Pad1) -> ROW3
- D11 pad 1: Net-(D11-Pad1) -> ROW4
- D12 pad 1: Net-(D12-Pad1) -> ROW5
- D13 pad 1: Net-(D13-Pad1) -> ROW0
- D14 pad 1: Net-(D14-Pad1) -> ROW1
- D15 pad 1: Net-(D15-Pad1) -> ROW2
- D16 pad 1: Net-(D16-Pad1) -> ROW3
- D17 pad 1: Net-(D17-Pad1) -> ROW4
- D18 pad 1: Net-(D18-Pad1) -> ROW5
- D19 pad 1: Net-(D19-Pad1) -> ROW0
- D2 pad 1: Net-(D2-Pad1) -> ROW1
- D20 pad 1: Net-(D20-Pad1) -> ROW1
- D21 pad 1: Net-(D21-Pad1) -> ROW2
- D22 pad 1: Net-(D22-Pad1) -> ROW3
- D23 pad 1: Net-(D23-Pad1) -> ROW4
- D25 pad 1: Net-(D25-Pad1) -> ROW0
- D26 pad 1: Net-(D26-Pad1) -> ROW1
- D27 pad 1: Net-(D27-Pad1) -> ROW2
- D28 pad 1: Net-(D28-Pad1) -> ROW3
- D29 pad 1: Net-(D29-Pad1) -> ROW4
- D3 pad 1: Net-(D3-Pad1) -> ROW2
- D31 pad 1: Net-(D31-Pad1) -> ROW0
- D32 pad 1: Net-(D32-Pad1) -> ROW1
- D33 pad 1: Net-(D33-Pad1) -> ROW2
- D332 pad 4: Net-(C331-Pad1) -> USB_5v
- D34 pad 1: Net-(D34-Pad1) -> ROW3
- D35 pad 1: Net-(D35-Pad1) -> ROW4
- D36 pad 1: Net-(D36-Pad1) -> ROW5
- D37 pad 1: Net-(D37-Pad1) -> ROW0
- D38 pad 1: Net-(D38-Pad1) -> ROW1
- D39 pad 1: Net-(D39-Pad1) -> ROW2
- D4 pad 1: Net-(D4-Pad1) -> ROW3
- D40 pad 1: Net-(D40-Pad1) -> ROW3
- D41 pad 1: Net-(D41-Pad1) -> ROW4
- D43 pad 1: Net-(D43-Pad1) -> ROW0
- D44 pad 1: Net-(D44-Pad1) -> ROW1
- D45 pad 1: Net-(D45-Pad1) -> ROW2
- D46 pad 1: Net-(D46-Pad1) -> ROW3
- D47 pad 1: Net-(D47-Pad1) -> ROW4
- D49 pad 1: Net-(D49-Pad1) -> ROW0
- D5 pad 1: Net-(D5-Pad1) -> ROW4
- D50 pad 1: Net-(D50-Pad1) -> ROW1
- D51 pad 1: Net-(D51-Pad1) -> ROW2
- D52 pad 1: Net-(D52-Pad1) -> ROW3
- D53 pad 1: Net-(D53-Pad1) -> ROW4
- D54 pad 1: Net-(D54-Pad1) -> ROW5
- D55 pad 1: Net-(D55-Pad1) -> ROW0
- D56 pad 1: Net-(D56-Pad1) -> ROW1
- D57 pad 1: Net-(D57-Pad1) -> ROW2
- D58 pad 1: Net-(D58-Pad1) -> ROW3
- D59 pad 1: Net-(D59-Pad1) -> ROW4
- D6 pad 1: Net-(D6-Pad1) -> ROW5
- D60 pad 1: Net-(D60-Pad1) -> ROW5
- D61 pad 1: Net-(D61-Pad1) -> ROW0
- D62 pad 1: Net-(D62-Pad1) -> ROW1
- D63 pad 1: Net-(D63-Pad1) -> ROW2
- D64 pad 1: Net-(D64-Pad1) -> ROW3
- D65 pad 1: Net-(D65-Pad1) -> ROW4
- D66 pad 1: Net-(D66-Pad1) -> ROW5
- D67 pad 1: Net-(D67-Pad1) -> ROW0
- D68 pad 1: Net-(D68-Pad1) -> ROW1
- D69 pad 1: Net-(D69-Pad1) -> ROW2
- D7 pad 1: Net-(D7-Pad1) -> ROW0
- D70 pad 1: Net-(D70-Pad1) -> ROW3
- D71 pad 1: Net-(D71-Pad1) -> ROW4
- D72 pad 1: Net-(D72-Pad1) -> ROW5
- D73 pad 1: Net-(D73-Pad1) -> ROW0
- D74 pad 1: Net-(D74-Pad1) -> ROW1
- D75 pad 1: Net-(D75-Pad1) -> ROW2
- D76 pad 1: Net-(D76-Pad1) -> ROW3
- D79 pad 1: Net-(D79-Pad1) -> ROW0
- D8 pad 1: Net-(D8-Pad1) -> ROW1
- D80 pad 1: Net-(D80-Pad1) -> ROW1
- D81 pad 1: Net-(D81-Pad1) -> ROW2
- D82 pad 1: Net-(D82-Pad1) -> ROW3
- D83 pad 1: Net-(D83-Pad1) -> ROW4
- D84 pad 1: Net-(D84-Pad1) -> ROW5
- D9 pad 1: Net-(D9-Pad1) -> ROW2
- U1 pad 42: ENC_B_1 -> ENC_B_2
Routing:
- net USB_5v: track 0.00 -> 4454.9 mm, vias 0 -> 26
- net COL14: track 0.00 -> 563.5 mm, vias 0 -> 9
- net COL13: track 0.00 -> 561.6 mm, vias 0 -> 9
- net ROW5: track 0.00 -> 519.7 mm, vias 0 -> 2
- net COL11: track 0.00 -> 510.7 mm, vias 0 -> 9
- net COL12: track 0.00 -> 488.5 mm, vias 0 -> 5
- net COL10: track 0.00 -> 481.3 mm, vias 0 -> 9
- net COL8: track 0.00 -> 466.4 mm, vias 0 -> 9
- net ROW3: track 0.00 -> 464.8 mm, vias 0 -> 2
- net COL9: track 0.00 -> 462.6 mm, vias 0 -> 7
- net ROW2: track 0.00 -> 448.9 mm
- net ROW4: track 0.00 -> 429.9 mm
- net COL6: track 0.00 -> 411.2 mm, vias 0 -> 8
- net COL7: track 0.00 -> 411.1 mm, vias 0 -> 8
- net ROW1: track 0.00 -> 403.8 mm, vias 0 -> 2
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- added copper zone on B.Cu, net USB_GND
- added copper zone on F.Cu, net USB_GND
Other:
- board size 403.9 x 129.5 mm -> 403.9 x 141.4 mm

Commit message: final commit (de momento)
Parts:
- added G007: LOGO, logo:jgfchj77eduardez, B.Cu at (319.4, 39.1)
Routing:
- net ROW2: track 448.9 -> 491.0 mm, vias 0 -> 4
- net USB_GND: track 23.3 -> 55.7 mm, vias 92 -> 249
Other:
- board size 403.9 x 141.4 mm -> 403.9 x 132.1 mm
