File: OLEDU_KiCad/OLEDUKEY/Key_matrix.sch (KiCad schematic (older format))
At the start: 168 parts, among them SW1 SW_Push, SW10 SW_Push, SW11 SW_Push, SW12 SW_Push, SW13 SW_Push, SW14 SW_Push, SW15 SW_Push, SW16 SW_Push, SW17 SW_Push, SW18 SW_Push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

Commit message: production files added
Connections:
- wire segments 457 -> 550
