File: OLEDU_KiCad/OLEDUKEY/RGB_Keys.sch (KiCad schematic (older format))
At the start: 212 parts, among them J301 Conn_01x03, J701 Conn_01x03, U301 74LVC1G125, U701 74LVC1G125

Commit message: pcb no copper
Parts:
- D301, D302, D303, D304, D305, D306, D307, D308, D309, D310, D311, D312, D313, D314, D315, D316, D317, D318, D319, D320, D321, D322, D323, D324, D325, D326, D327, D328, D329, D330, D331, D332, D333, D334, D335, D336, D337, D338, D339, D340, D341, D342, D343, D344, D345, D346, D347, D348, D349, D350, D351, D352, D353, D354, D355, D356, D357, D358, D359, D360, D361, D362, D363, D364, D365, D366, D367, D368, D369, D370, D371, D372, D373, D374, D375, D376, D377, D378, D379, D380, D381, D382, D383, D384, D385, D386: footprint Keebio-Parts:SK6812-MINI-E -> LED_SDM_MOD:SK6812-MINI-E
- D701, D702, D703, D704, D705, D706, D707, D708, D709, D710, D711, D712, D713, D714, D715, D716, D717, D718: footprint LED_SMD:LED_SK6812MINI_PLCC4_3.5x3.5mm_P1.75mm -> LED_SDM_MOD:LED_SK6812MINI_PLCC4_3.5x3.5mm_P1.75mm

Commit message: production files added
Connections:
- wire segments 1384 -> 1395
Changed lines of the file:
@@
 	10250 5450 10850 5450
-Wire Wire Line
-	10850 4150 10850 4400
 Wire Wire Line
 	10850 4900 10850 5450
@@
 Wire Wire Line
 	22600 1850 24000 1850
-Wire Wire Line
-	10850 4500 10850 4550
 Connection ~ 1000 4550
 Wire Wire Line
@@
 	6350 12500 6400 12500
 Wire Wire Line
-	6650 14000 6650 13650
-Wire Wire Line
 	6400 14000 6650 14000
 Wire Wire Line
@@
 Connection ~ 4050 10950
 Wire Wire Line
-	5250 14000 5250 13250
-Wire Wire Line
 	5050 14000 5100 14000
 Connection ~ 5100 14000
@@
 Connection ~ 5250 13250
 Wire Wire Line
-	5250 13250 5250 12500
+	5250 13250 5250 12900
 Connection ~ 5100 13250
 Wire Wire Line
@@
 Connection ~ 5250 12500
 Wire Wire Line
-	5250 12500 5250 11750
+	5250 12500 5250 12150
 Connection ~ 5100 12500
 Wire Wire Line
@@
 $EndComp
 Wire Wire Line
-	4600 12150 5300 12150
-Wire Wire Line
-	4600 12900 5300 12900
-Wire Wire Line
-	4600 13650 5300 13650
-Wire Wire Line
 	4600 14400 5300 14400
 Wire Wire Line
@@
 Wire Wire Line
 	2000 1850 2000 2650
+Wire Wire Line
+	2800 14400 2800 14000
+Connection ~ 2800 14000
+Wire Wire Line
+	4050 14400 4050 14000
+Wire Wire Line
+	10850 4500 10850 4550
+Wire Wire Line
+	10850 4150 10850 4550
+Connection ~ 4050 14000
+Wire Wire Line
+	5300 14400 5300 14000
+Wire Wire Line
+	5300 14000 5250 14000
+Connection ~ 5250 14000
+Wire Wire Line
+	5250 13250 5250 13650
+Wire Wire Line
+	4600 13650 5250 13650
+Connection ~ 5250 13650
+Wire Wire Line
+	5250 13650 5250 14000
+Wire Wire Line
+	5250 13650 5300 13650
+Wire Wire Line
+	4600 12900 5250 12900
+Connection ~ 5250 12900
+Wire Wire Line
+	5250 12900 5250 12500
+Wire Wire Line
+	5250 12900 5300 12900
+Wire Wire Line
+	6650 13650 6650 14000
+Connection ~ 6650 14000
+Wire Wire Line
+	6650 14000 6650 14400
+Wire Wire Line
+	4600 12150 5250 12150
+Connection ~ 5250 12150
+Wire Wire Line
+	5250 12150 5250 11750
+Wire Wire Line
+	5250 12150 5300 12150
 $EndSCHEMATC
